File: pcb/hand_cluster.kicad_pcb (KiCad board)
At the start: 2 copper layers, 0 parts

Commit message: Designed the version of a plaid modular hand cluster
Parts:
- added DA1: 1N4148, Diode_THT:D_DO-35_SOD27_P7.62mm_Horizontal, F.Cu at (168.7, -51.1)
- added DA2: 1N4148, Diode_THT:D_DO-35_SOD27_P7.62mm_Horizontal, F.Cu at (178.8, -51.1)
- added DA3: 1N4148, Diode_THT:D_DO-35_SOD27_P7.62mm_Horizontal, F.Cu at (189.0, -51.1)
- added DA4: 1N4148, Diode_THT:D_DO-35_SOD27_P7.62mm_Horizontal, F.Cu at (199.8, -51.1)
- added DA5: 1N4148, Diode_THT:D_DO-35_SOD27_P7.62mm_Horizontal, F.Cu at (210.0, -51.1)
- added DA6: 1N4148, Diode_THT:D_DO-35_SOD27_P7.62mm_Horizontal, F.Cu at (220.1, -51.1)
- added DA7: 1N4148, Diode_THT:D_DO-35_SOD27_P7.62mm_Horizontal, F.Cu at (230.3, -51.1)
- added DB1: 1N4148, Diode_THT:D_DO-35_SOD27_P7.62mm_Horizontal, F.Cu at (171.2, -49.2)
- added DB2: 1N4148, Diode_THT:D_DO-35_SOD27_P7.62mm_Horizontal, F.Cu at (181.4, -49.2)
- added DB3: 1N4148, Diode_THT:D_DO-35_SOD27_P7.62mm_Horizontal, F.Cu at (191.6, -49.2)
- added DB4: 1N4148, Diode_THT:D_DO-35_SOD27_P7.62mm_Horizontal, F.Cu at (202.3, -49.2)
- added DB5: 1N4148, Diode_THT:D_DO-35_SOD27_P7.62mm_Horizontal, F.Cu at (212.5, -49.2)
- added DB6: 1N4148, Diode_THT:D_DO-35_SOD27_P7.62mm_Horizontal, F.Cu at (222.7, -49.2)
- added DB7: 1N4148, Diode_THT:D_DO-35_SOD27_P7.62mm_Horizontal, F.Cu at (232.8, -49.2)
- added DC1: 1N4148, Diode_THT:D_DO-35_SOD27_P7.62mm_Horizontal, F.Cu at (173.8, -47.3)
- added DC2: 1N4148, Diode_THT:D_DO-35_SOD27_P7.62mm_Horizontal, F.Cu at (183.9, -47.3)
- added DC3: 1N4148, Diode_THT:D_DO-35_SOD27_P7.62mm_Horizontal, F.Cu at (194.1, -47.3)
- added DC4: 1N4148, Diode_THT:D_DO-35_SOD27_P7.62mm_Horizontal, F.Cu at (204.9, -47.3)
- added DC5: 1N4148, Diode_THT:D_DO-35_SOD27_P7.62mm_Horizontal, F.Cu at (215.0, -47.3)
- added DC6: 1N4148, Diode_THT:D_DO-35_SOD27_P7.62mm_Horizontal, F.Cu at (225.2, -47.3)
- added DC7: 1N4148, Diode_THT:D_DO-35_SOD27_P7.62mm_Horizontal, F.Cu at (235.4, -47.3)
- added DD1: 1N4148, Diode_THT:D_DO-35_SOD27_P7.62mm_Horizontal, F.Cu at (176.3, -45.4)
- added DD2: 1N4148, Diode_THT:D_DO-35_SOD27_P7.62mm_Horizontal, F.Cu at (186.5, -45.4)
- added DD3: 1N4148, Diode_THT:D_DO-35_SOD27_P7.62mm_Horizontal, F.Cu at (196.6, -45.4)
- added DD4: 1N4148, Diode_THT:D_DO-35_SOD27_P7.62mm_Horizontal, F.Cu at (207.4, -45.4)
- added DD5: 1N4148, Diode_THT:D_DO-35_SOD27_P7.62mm_Horizontal, F.Cu at (217.6, -45.4)
- added DD6: 1N4148, Diode_THT:D_DO-35_SOD27_P7.62mm_Horizontal, F.Cu at (227.7, -45.4)
- added DD7: 1N4148, Diode_THT:D_DO-35_SOD27_P7.62mm_Horizontal, F.Cu at (237.9, -45.4)
- added J1: AudioJack4, Keebio-Parts:TRRS-PJ-320A-dual-labeled, F.Cu at (262.3, -58.4)
- added J2: AudioJack4, Keebio-Parts:TRRS-PJ-320A-dual-labeled, F.Cu at (253.2, -58.4)
- added JM1.1: Conn_01x07_Male, Connector_PinHeader_2.54mm:PinHeader_1x07_P2.54mm_Vertical, F.Cu at (241.7, -53.1)
- added JM1.2: Conn_01x07_Male, Connector_PinHeader_2.54mm:PinHeader_1x07_P2.54mm_Vertical, F.Cu at (164.9, -53.1)
- added R1: 2.2k, Keebio-Parts:Resistor, F.Cu at (255.3, -42.6)
- added R2: 2.2k, Keebio-Parts:Resistor, F.Cu at (255.4, -39.9)
- added REF**: MountingHole_3.2mm_M3, MountingHole:MountingHole_3.2mm_M3, F.Cu at (274.0, -30.1)
- added REF**: MountingHole_3.2mm_M3, MountingHole:MountingHole_3.2mm_M3, F.Cu at (227.7, 44.9)
- added REF**: MountingHole_3.2mm_M3, MountingHole:MountingHole_3.2mm_M3, F.Cu at (274.0, -1.10)
- added REF**: MountingHole_3.2mm_M3, MountingHole:MountingHole_3.2mm_M3, F.Cu at (274.0, -57.1)
- added REF**: MountingHole_3.2mm_M3, MountingHole:MountingHole_3.2mm_M3, F.Cu at (122.7, -57.1)
- added REF**: MountingHole_3.2mm_M3, MountingHole:MountingHole_3.2mm_M3, F.Cu at (122.7, -30.1)
- added REF**: MountingHole_3.2mm_M3, MountingHole:MountingHole_3.2mm_M3, F.Cu at (122.7, 44.9)
- added SWA1: Cherry MX, acerne:Hybrid_Plate_150H_Dual_hole-nosilk, F.Cu at (141.0, -25.7)
- added SWA2: Cherry MX, Keebio-Parts:Hybrid_Plate_100H_Dual_hole-nosilk, F.Cu at (165.1, -25.7)
- added SWA3: Cherry MX, Keebio-Parts:Hybrid_Plate_100H_Dual_hole-nosilk, F.Cu at (184.2, -25.7)
- added SWA4: Cherry MX, Keebio-Parts:Hybrid_Plate_100H_Dual_hole-nosilk, F.Cu at (203.2, -25.7)
- added SWA5: Cherry MX, Keebio-Parts:Hybrid_Plate_100H_Dual_hole-nosilk, F.Cu at (222.3, -25.7)
- added SWA6: Cherry MX, Keebio-Parts:Hybrid_Plate_100H_Dual_hole-nosilk, F.Cu at (241.3, -25.7)
- added SWA7.1: Cherry MX, Keebio-Parts:Hybrid_Plate_100H_Dual_hole-nosilk, F.Cu at (260.4, -25.7)
- added SWB1: Cherry MX, acerne:Hybrid_Plate_150H_Dual_hole-nosilk, F.Cu at (141.0, -6.66)
- added SWB2: Cherry MX, Keebio-Parts:Hybrid_Plate_100H_Dual_hole-nosilk, F.Cu at (165.1, -6.66)
- added SWB3: Cherry MX, Keebio-Parts:Hybrid_Plate_100H_Dual_hole-nosilk, F.Cu at (184.2, -6.66)
- added SWB4: Cherry MX, Keebio-Parts:Hybrid_Plate_100H_Dual_hole-nosilk, F.Cu at (203.2, -6.66)
- added SWB5: Cherry MX, Keebio-Parts:Hybrid_Plate_100H_Dual_hole-nosilk, F.Cu at (222.3, -6.66)
- added SWB6: Cherry MX, Keebio-Parts:Hybrid_Plate_100H_Dual_hole-nosilk, F.Cu at (241.3, -6.66)
- added SWC1: Cherry MX, acerne:Hybrid_Plate_150H_Dual_hole-nosilk, F.Cu at (141.0, 12.4)
- added SWC2: Cherry MX, Keebio-Parts:Hybrid_Plate_100H_Dual_hole-nosilk, F.Cu at (165.1, 12.4)
- added SWC3: Cherry MX, Keebio-Parts:Hybrid_Plate_100H_Dual_hole-nosilk, F.Cu at (184.2, 12.4)
- added SWC4: Cherry MX, Keebio-Parts:Hybrid_Plate_100H_Dual_hole-nosilk, F.Cu at (203.2, 12.4)
- added SWC5: Cherry MX, Keebio-Parts:Hybrid_Plate_100H_Dual_hole-nosilk, F.Cu at (222.3, 12.4)
- added SWC6: Cherry MX, Keebio-Parts:Hybrid_Plate_100H_Dual_hole-nosilk, F.Cu at (241.3, 12.4)
- added SWD1: Cherry MX, acerne:Hybrid_Plate_150H_Dual_hole-nosilk, F.Cu at (141.0, 31.4)
- added SWD2.1: Cherry MX, Keebio-Parts:Hybrid_Plate_100H_Dual_hole-nosilk, F.Cu at (165.1, 31.4)
- added SWD2.2: Cherry MX, Keebio-Parts:Hybrid_Plate_100H_Dual_hole-nosilk, F.Cu at (174.7, 31.4)
- added SWD3.1: Cherry MX, Keebio-Parts:Hybrid_Plate_100H_Dual_hole-nosilk, F.Cu at (184.2, 31.4)
- added SWD3.2: Cherry MX, Keebio-Parts:Hybrid_Plate_100H_Dual_hole-nosilk, F.Cu at (193.7, 31.4)
- added SWD4.1: Cherry MX, Keebio-Parts:Hybrid_Plate_100H_Dual_hole-nosilk, F.Cu at (203.2, 31.4)
- added SWD4.2: Cherry MX, Keebio-Parts:Hybrid_Plate_100H_Dual_hole-nosilk, F.Cu at (212.8, 31.4)
- added SWD5: Cherry MX, Keebio-Parts:Hybrid_Plate_100H_Dual_hole-nosilk, F.Cu at (222.3, 31.4)
- added SWD6.1: Cherry MX, Keebio-Parts:Hybrid_Plate_100H_Dual_hole-nosilk, F.Cu at (260.4, -6.66)
- added SWD6.2: Cherry MX, Keebio-Parts:Hybrid_Plate_100H_Dual_hole-nosilk, F.Cu at (260.4, -16.2)
- added SWRST1: SW_Push, Button_Switch_THT:SW_PUSH_6mm, F.Cu at (268.2, -43.9)
- added U1: ProMicro, Keebio-Parts:ArduinoProMicro, F.Cu at (142.5, -45.4)
Routing:
- net SDA: track 0.00 -> 307.3 mm
- net SCL: track 0.00 -> 302.4 mm
- net Col6: track 0.00 -> 275.0 mm
- net Net-(DA1-Pad2): track 0.00 -> 221.4 mm
- net Col5: track 0.00 -> 207.0 mm
- net VCC: track 0.00 -> 202.6 mm
- net Net-(DB1-Pad2): track 0.00 -> 200.7 mm
- net Col4: track 0.00 -> 195.0 mm
- net Net-(DC1-Pad2): track 0.00 -> 191.5 mm
- net Col3: track 0.00 -> 174.7 mm
- net Reset: track 0.00 -> 162.7 mm
- net Net-(DD1-Pad2): track 0.00 -> 155.9 mm
- net Col7: track 0.00 -> 144.7 mm
- net RowC: track 0.00 -> 130.8 mm
- net RowD: track 0.00 -> 102.7 mm
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- added copper zone on F.Cu, net GND
Other:
- board outline added: 159.2 x 110 mm
- net class Default: clearance 0.2 -> 0.5; trace_width 0.25 -> 0.5
- net class Large added: clearance 0.5, trace_width 0.5, via_dia 0.8, via_drill 0.4
- rule pad_to_mask_clearance: 0.051 -> 0.5
- rule trace_clearance: 0.2 -> 0.5
